File: nerdqaxe++/nerdqaxe++/level_shifter.kicad_sch (KiCad schematic)
At the start: 21 parts, among them U17 TLV3544

Commit message: Rev7 complete
Parts:
- R67: PARTNO (none) -> RC0402JR-070RL; now not fitted
Changed lines of the file:
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@@
 		(on_board yes)
 		(in_pos_files yes)
-		(dnp no)
+		(dnp yes)
 		(fields_autoplaced yes)
 		(property "Reference" "R67"
@@
 			(hide yes)
 			(show_name no)
+			(do_not_autoplace no)
+			(effects
+				(font
+					(size 1.27 1.27)
+				)
+			)
+		)
+		(property "PARTNO" "RC0402JR-070RL"
+			(at 140.97 38.1 90)
+			(hide yes)
+			(show_name no)
